Commit message: Add FV and integrate launch file

File: models/FV/f1.xacro (robot description, xacro)
@@ -1,8 +1,8 @@
 <?xml version="1.0" ?>
-<robot name="LV" xmlns:xacro="http://www.ros.org/wiki/xacro">
-  <xacro:include filename="$(find platooning_tracking_gazebo)/models/LV/model.gazebo" />
+<robot name="FV" xmlns:xacro="http://www.ros.org/wiki/xacro">
+  <xacro:include filename="$(find platooning_tracking_gazebo)/models/FV/f1.gazebo" />
   <joint name="chassis" type="fixed">
-    <parent link="LV__link_0"/>
-    <child link="LV__link_1"/>
+    <parent link="FV__link_0"/>
+    <child link="FV__link_1"/>
     <origin rpy="0  0  0" xyz="0      -0.19568  0.03714"/>
     <axis xyz="0  1  0"/>
@@ -11,34 +11,42 @@
   </joint>
   <!-- front  -->
-  <joint name="front_left" type="continuous">
-    <parent link="LV__link_0"/>
-    <child link="LV__link_2_clone_0_clone"/>
+  <joint name="f1_front_left" type="continuous">
+    <parent link="FV__link_0"/>
+    <child link="FV__link_2_clone_0_clone"/>
     <origin rpy="0      1.5707  0" xyz="-0.11     0.39431 -0.03785"/>
     <axis xyz="0   0   -1"/>
 	<limit effort="10.0" velocity="100.0"/>
   </joint>
-  <joint name="front_right" type="continuous">
-    <parent link="LV__link_0"/>
-    <child link="LV__link_2_clone"/>
+  <joint name="f1_front_right" type="continuous">
+    <parent link="FV__link_0"/>
+    <child link="FV__link_2_clone"/>
     <origin rpy="0      1.5707  0" xyz="0.11     0.39431 -0.03785"/>
 	<axis xyz="0   0   -1"/>
     <limit effort="10.0" velocity="100.0"/>
   </joint>
+  <!-- lidar -->
+  <joint name="lidar" type="revolute">
+    <parent link="FV__link_0"/>
+    <child link="laser"/>
+    <origin rpy="0  0  0" xyz="0       0.41413  0.08635"/>
+    <axis xyz="1  0  0"/>
+    <limit effort="-1.0" lower="-1.79769e+308" upper="1.79769e+308" velocity="-1.0"/>
+  </joint>
   <!-- rear -->
-  <joint name="rear_left" type="continuous">
-    <parent link="LV__link_1"/>
-    <child link="LV__link_2_clone_0"/>
+  <joint name="f1_rear_left" type="continuous">
+    <parent link="FV__link_1"/>
+    <child link="FV__link_2_clone_0"/>
     <origin rpy="0      1.5707  0" xyz="-0.11  -0.51  -0.075"/>
     <axis xyz="0   0   1"/>
     <limit effort="10.0" velocity="100.0"/>
   </joint>
-  <joint name="rear_right" type="continuous">
-    <parent link="LV__link_1"/>
-    <child link="LV__link_2_clone_1"/>
+  <joint name="f1_rear_right" type="continuous">
+    <parent link="FV__link_1"/>
+    <child link="FV__link_2_clone_1"/>
     <origin rpy="0      1.5707  0" xyz="0.11  -0.51  -0.075"/>
     <axis xyz="0   0   1"/>
     <limit effort="10.0" velocity="100.0"/>
   </joint>
-  <link name="LV__link_0">
+  <link name="FV__link_0">
     <inertial>
       <mass value="1"/>
@@ -46,5 +54,5 @@
       <inertia ixx="0.166667" ixy="0" ixz="0" iyy="0.166667" iyz="0" izz="0.166667"/>
     </inertial>
-    <collision name="LV__collision">
+    <collision name="FV__collision">
       <origin rpy="0  0  0" xyz="0       0.40431  0.00714"/>
       <geometry>
@@ -52,5 +60,5 @@
       </geometry>
     </collision>
-    <visual name="LV__visual">
+    <visual name="FV__visual">
       <origin rpy="0  0  0" xyz="0       0.40431  0.00714"/>
       <geometry>
@@ -59,5 +67,5 @@
     </visual>
   </link>
-  <link name="LV__link_1">
+  <link name="FV__link_1">
     <inertial>
       <mass value="1"/>
@@ -65,5 +73,5 @@
       <inertia ixx="0.166667" ixy="0" ixz="0" iyy="0.166667" iyz="0" izz="0.166667"/>
     </inertial>
-    <collision name="LV__collision">
+    <collision name="FV__collision">
       <origin rpy="0  0  0" xyz="0  0  0"/>
       <geometry>
@@ -71,5 +79,5 @@
       </geometry>
     </collision>
-    <visual name="LV__visual">
+    <visual name="FV__visual">
       <origin rpy="0  0  0" xyz="0  0  0"/>
       <geometry>
@@ -78,5 +86,5 @@
     </visual>
   </link>
-  <link name="LV__link_2_clone">
+  <link name="FV__link_2_clone">
     <inertial>
       <mass value="1"/>
@@ -84,5 +92,5 @@
       <inertia ixx="0.145833" ixy="0" ixz="0" iyy="0.145833" iyz="0" izz="0.125"/>
     </inertial>
-    <collision name="LV__collision">
+    <collision name="FV__collision">
       <origin rpy="0  0  0" xyz="0  0  0"/>
       <geometry>
@@ -90,5 +98,5 @@
       </geometry>
     </collision>
-    <visual name="LV__visual">
+    <visual name="FV__visual">
       <origin rpy="0  0  0" xyz="0  0  0"/>
       <geometry>
@@ -97,5 +105,5 @@
     </visual>
   </link>
-  <link name="LV__link_2_clone_0">
+  <link name="FV__link_2_clone_0">
     <inertial>
       <mass value="1"/>
@@ -103,5 +111,5 @@
       <inertia ixx="0.145833" ixy="0" ixz="0" iyy="0.145833" iyz="0" izz="0.125"/>
     </inertial>
-    <collision name="LV__collision">
+    <collision name="FV__collision">
       <origin rpy="0  0  0" xyz="0  0  0"/>
       <geometry>
@@ -109,5 +117,5 @@
       </geometry>
     </collision>
-    <visual name="LV__visual">
+    <visual name="FV__visual">
       <origin rpy="0  0  0" xyz="0  0  0"/>
       <geometry>
@@ -116,5 +124,5 @@
     </visual>
   </link>
-  <link name="LV__link_2_clone_0_clone">
+  <link name="FV__link_2_clone_0_clone">
     <inertial>
       <mass value="1"/>
@@ -122,5 +130,5 @@
       <inertia ixx="0.145833" ixy="0" ixz="0" iyy="0.145833" iyz="0" izz="0.125"/>
     </inertial>
-    <collision name="LV__collision">
+    <collision name="FV__collision">
       <origin rpy="0  0  0" xyz="0  0  0"/>
       <geometry>
@@ -128,5 +136,5 @@
       </geometry>
     </collision>
-    <visual name="LV__visual">
+    <visual name="FV__visual">
       <origin rpy="0  0  0" xyz="0  0  0"/>
       <geometry>
@@ -135,5 +143,5 @@
     </visual>
   </link>
-  <link name="LV__link_2_clone_1">
+  <link name="FV__link_2_clone_1">
     <inertial>
       <mass value="1"/>
@@ -141,5 +149,5 @@
       <inertia ixx="0.145833" ixy="0" ixz="0" iyy="0.145833" iyz="0" izz="0.125"/>
     </inertial>
-    <collision name="LV__collision">
+    <collision name="FV__collision">
       <origin rpy="0  0  0" xyz="0  0  0"/>
       <geometry>
@@ -147,5 +155,5 @@
       </geometry>
     </collision>
-    <visual name="LV__visual">
+    <visual name="FV__visual">
       <origin rpy="0  0  0" xyz="0  0  0"/>
       <geometry>
@@ -154,7 +162,20 @@
     </visual>
   </link>
+  <link name="laser">
+    <inertial>
+      <mass value="0.1"/>
+      <origin rpy="0  0  0" xyz="0  0  0"/>
+      <inertia ixx="0" ixy="0" ixz="0" iyy="0" iyz="0" izz="0"/>
+    </inertial>
+    <visual name="FV__visual">
+      <origin rpy="0  0  0" xyz="0  0  0"/>
+      <geometry>
+        <mesh filename="package://rrbot_description/meshes/hokuyo.dae" scale="1.0 1.0 1.0"/>
+      </geometry>
+    </visual>
+  </link>
   <transmission name="tran1">
     <type>transmission_interface/SimpleTransmission</type>
-    <joint name="front_left">
+    <joint name="f1_front_left">
       <hardwareInterface>hardware_interface/EffortJointInterface</hardwareInterface>
     </joint>
@@ -166,5 +187,5 @@
   <transmission name="tran2">
     <type>transmission_interface/SimpleTransmission</type>
-    <joint name="front_right">
+    <joint name="f1_front_right">
       <hardwareInterface>hardware_interface/EffortJointInterface</hardwareInterface>
     </joint>

File: models/LV/model_backup.xacro (robot description, xacro)
@@ -2,42 +2,41 @@
 <robot name="LV" xmlns:xacro="http://www.ros.org/wiki/xacro">
   <xacro:include filename="$(find platooning_tracking_gazebo)/models/LV/model.gazebo" />
-  <joint name="chassis" type="fixed">
-    <parent link="LV__link_0"/>
-    <child link="LV__link_1"/>
-    <origin rpy="0  0  0" xyz="0      -0.19568  0.03714"/>
-    <axis xyz="0  1  0"/>
-    <!--limit effort="-1.0" lower="-1.79769e+308" upper="1.79769e+308" velocity="-1.0"/-->
-    <limit effort="10.0" velocity="100.0"/>
-  </joint>
-  <!-- front  -->
+  <xacro:include filename="$(find platooning_tracking_gazebo)/models/LV/materials.xacro" />
+  <!-- Joint -->
+  <!-- front -->
   <joint name="front_left" type="continuous">
     <parent link="LV__link_0"/>
-    <child link="LV__link_2_clone_0_clone"/>
-    <origin rpy="0      1.5707  0" xyz="-0.11     0.39431 -0.03785"/>
-    <axis xyz="0   0   -1"/>
-	<limit effort="10.0" velocity="100.0"/>
+    <child link="LV__link_1_clone"/>
+    <origin rpy="0      1.5707  0" xyz="-0.06999  0.51724 -0.039"/>
+    <axis xyz="0 0 -1"/>
+    <dynamics damping="0.7"/>
+    <limit effort="100" velocity="100"/>
   </joint>
   <joint name="front_right" type="continuous">
     <parent link="LV__link_0"/>
-    <child link="LV__link_2_clone"/>
-    <origin rpy="0      1.5707  0" xyz="0.11     0.39431 -0.03785"/>
-	<axis xyz="0   0   -1"/>
-    <limit effort="10.0" velocity="100.0"/>
+    <child link="LV__link_1_clone_0"/>
+    <origin rpy="0      1.5707  0" xyz="0.06999  0.51441 -0.039"/>
+    <axis xyz="0 0 -1"/>
+    <dynamics damping="0.7"/>
+    <limit effort="100" velocity="100"/>
   </joint>
   <!-- rear -->
   <joint name="rear_left" type="continuous">
-    <parent link="LV__link_1"/>
-    <child link="LV__link_2_clone_0"/>
-    <origin rpy="0      1.5707  0" xyz="-0.11  -0.51  -0.075"/>
-    <axis xyz="0   0   1"/>
-    <limit effort="10.0" velocity="100.0"/>
+    <parent link="LV__link_0"/>
+    <child link="LV__link_1"/>
+    <origin rpy="0      1.5707  0" xyz="-0.06999 -0.53055 -0.039"/>
+    <axis xyz="0 0 -1"/>
+    <dynamics damping="0.7"/>
+    <limit effort="10" velocity="100"/>
   </joint>
   <joint name="rear_right" type="continuous">
-    <parent link="LV__link_1"/>
-    <child link="LV__link_2_clone_1"/>
-    <origin rpy="0      1.5707  0" xyz="0.11  -0.51  -0.075"/>
-    <axis xyz="0   0   1"/>
-    <limit effort="10.0" velocity="100.0"/>
+    <parent link="LV__link_0"/>
+    <child link="LV__link_1_clone_1"/>
+    <origin rpy="0      1.5707  0" xyz="0.06999 -0.53055 -0.039"/>
+    <axis xyz="0 0 -1"/>
+    <dynamics damping="0.7"/>
+    <limit effort="10" velocity="100"/>
   </joint>
+  <!-- Link -->
   <link name="LV__link_0">
     <inertial>
@@ -47,36 +46,17 @@
     </inertial>
     <collision name="LV__collision">
-      <origin rpy="0  0  0" xyz="0       0.40431  0.00714"/>
+      <origin rpy="0  0  0" xyz="0       0.02944  0.156"/>
       <geometry>
-        <box size="0.18 0.1 0.13"/>
+        <box size="0.18 1.2 0.35"/>
       </geometry>
     </collision>
     <visual name="LV__visual">
-      <origin rpy="0  0  0" xyz="0       0.40431  0.00714"/>
+      <origin rpy="0  0  0" xyz="0       0.02944  0.156"/>
       <geometry>
-        <box size="0.18 0.1 0.13"/>
+        <box size="0.18 1.2 0.35"/>
       </geometry>
     </visual>
   </link>
   <link name="LV__link_1">
-    <inertial>
-      <mass value="1"/>
-      <origin rpy="0  0  0" xyz="0  0  0"/>
-      <inertia ixx="0.166667" ixy="0" ixz="0" iyy="0.166667" iyz="0" izz="0.166667"/>
-    </inertial>
-    <collision name="LV__collision">
-      <origin rpy="0  0  0" xyz="0  0  0"/>
-      <geometry>
-        <box size="0.18 1.1 0.19"/>
-      </geometry>
-    </collision>
-    <visual name="LV__visual">
-      <origin rpy="0  0  0" xyz="0  0  0"/>
-      <geometry>
-        <box size="0.18 1.1 0.19"/>
-      </geometry>
-    </visual>
-  </link>
-  <link name="LV__link_2_clone">
     <inertial>
       <mass value="1"/>
@@ -97,5 +77,5 @@
     </visual>
   </link>
-  <link name="LV__link_2_clone_0">
+  <link name="LV__link_1_clone">
     <inertial>
       <mass value="1"/>
@@ -116,5 +96,5 @@
     </visual>
   </link>
-  <link name="LV__link_2_clone_0_clone">
+  <link name="LV__link_1_clone_0">
     <inertial>
       <mass value="1"/>
@@ -135,5 +115,5 @@
     </visual>
   </link>
-  <link name="LV__link_2_clone_1">
+  <link name="LV__link_1_clone_1">
     <inertial>
       <mass value="1"/>

Commit message: Add FV, LV, test, duckietown world

File: models/FV/f1.xacro (robot description, xacro)
@@ -28,5 +28,5 @@
   <joint name="lidar" type="revolute">
     <parent link="FV__link_0"/>
-    <child link="laser"/>
+    <child link="hokuyo"/>
     <origin rpy="0  0  0" xyz="0       0.41413  0.08635"/>
     <axis xyz="1  0  0"/>
@@ -162,5 +162,5 @@
     </visual>
   </link>
-  <link name="laser">
+  <link name="hokuyo">
     <inertial>
       <mass value="0.1"/>
